File: pcb/indigo.kicad_pcb (KiCad board)
At the start: 2 copper layers, 96 parts, among them SW1 SW_Push, SW10 SW_Push, SW11 SW_Push, SW12 SW_Push, SW13 SW_Push, SW14 SW_Push, SW15 SW_Push, SW16 SW_Push, SW17 SW_Push, SW18 SW_Push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

Commit message: pcb, features
Parts:
- removed D18, D26, D34, D35, D36, D41, D42, D43, D44, D49, D50, D51, D52, D57, D58, D59, D60, D65, D66, D67, D68: D, Keebio-Parts:Diode-Hybrid-Back
- removed D19, D20, D27, D28: WS2812B, LED_SMD:LED_WS2812B_PLCC4_5.0x5.0mm_P3.2mm
- removed the D29 at (241.3, 121.9)
- removed the D30 at (241.3, 121.9)
- added D10: WS2812B, LED_SMD:LED_WS2812B_PLCC4_5.0x5.0mm_P3.2mm, B.Cu at (66.7, 123.8)
- added D11: WS2812B, LED_SMD:LED_WS2812B_PLCC4_5.0x5.0mm_P3.2mm, F.Cu at (119.1, 123.8)
- added D32: D, Keebio-Parts:Diode-dual, F.Cu at (128.6, 123.8)
- added J1: Conn_01x04, Connector_PinHeader_2.54mm:PinHeader_1x04_P2.54mm_Vertical, F.Cu at (221.3, 103.5)
- added R1: R, Keebio-Parts:Resistor-Hybrid, F.Cu at (217.5, 107.4)
- added R2: R, Keebio-Parts:Resistor-Hybrid-Back, F.Cu at (217.5, 107.4)
- added R3: R, Keebio-Parts:Resistor-Hybrid, F.Cu at (214.9, 107.4)
- added R4: R, Keebio-Parts:Resistor-Hybrid-Back, F.Cu at (214.9, 107.4)
- added SW10: SW_Push, Keebio-Parts:Hybrid_PCB_100H_Dual_hole-nosilk, F.Cu at (138.1, 123.8)
- D13, D14, D15, D23, D37, D38, D39, D40, D45, D46, D47, D48, D53, D54, D55, D56, D61, D62, D63, D64: footprint Keebio-Parts:Diode-Hybrid-Back -> Keebio-Parts:Diode-dual
- D16: value D -> WS2812B; footprint Keebio-Parts:Diode-Hybrid-Back -> LED_SMD:LED_WS2812B_PLCC4_5.0x5.0mm_P3.2mm; moved to F.Cu
- D17, D22: value D -> WS2812B; footprint Keebio-Parts:Diode-Hybrid-Back -> LED_SMD:LED_WS2812B_PLCC4_5.0x5.0mm_P3.2mm
- D21: value D -> WS2812B; footprint Keebio-Parts:Diode-Hybrid-Back -> LED_SMD:LED_WS2812B_PLCC4_5.0x5.0mm_P3.2mm; moved to B.Cu
- D24, D25: footprint Keebio-Parts:Diode-Hybrid-Back -> Keebio-Parts:Diode-dual; moved to F.Cu
- D29: renamed from D31; footprint Keebio-Parts:Diode-Hybrid-Back -> Keebio-Parts:Diode-dual
- D30: renamed from D32; footprint Keebio-Parts:Diode-Hybrid-Back -> Keebio-Parts:Diode-dual
- D31: renamed from D33; footprint Keebio-Parts:Diode-Hybrid-Back -> Keebio-Parts:Diode-dual
- SW1, SW2, SW3, SW4, SW5, SW6, SW7, SW8, SW9: footprint Keebio-Parts:Hybrid_PCB_100H_Dual_hole -> Keebio-Parts:Hybrid_PCB_100H_Dual_hole-nosilk
- SW11: renamed from SW10; footprint Keebio-Parts:Hybrid_PCB_100H_Dual_hole -> Keebio-Parts:Hybrid_PCB_100H_Dual_hole-nosilk
- SW12: renamed from SW11; footprint Keebio-Parts:Hybrid_PCB_100H_Dual_hole -> Keebio-Parts:Hybrid_PCB_100H_Dual_hole-nosilk
- SW13: renamed from SW12; footprint Keebio-Parts:Hybrid_PCB_100H_Dual_hole -> Keebio-Parts:Hybrid_PCB_100H_Dual_hole-nosilk
- SW14: renamed from SW13; footprint Keebio-Parts:Hybrid_PCB_100H_Dual_hole -> Keebio-Parts:Hybrid_PCB_100H_Dual_hole-nosilk
- SW15: renamed from SW14; footprint Keebio-Parts:Hybrid_PCB_100H_Dual_hole -> Keebio-Parts:Hybrid_PCB_100H_Dual_hole-nosilk
- SW16: renamed from SW15; footprint Keebio-Parts:Hybrid_PCB_100H_Dual_hole -> Keebio-Parts:Hybrid_PCB_100H_Dual_hole-nosilk
- SW17: renamed from SW16; footprint Keebio-Parts:Hybrid_PCB_100H_Dual_hole -> Keebio-Parts:Hybrid_PCB_100H_Dual_hole-nosilk
- SW18: renamed from SW17; footprint Keebio-Parts:Hybrid_PCB_100H_Dual_hole -> Keebio-Parts:Hybrid_PCB_100H_Dual_hole-nosilk
- SW19: renamed from SW18; footprint Keebio-Parts:Hybrid_PCB_100H_Dual_hole -> Keebio-Parts:Hybrid_PCB_100H_Dual_hole-nosilk
- SW20: renamed from SW19; footprint Keebio-Parts:Hybrid_PCB_100H_Dual_hole -> Keebio-Parts:Hybrid_PCB_100H_Dual_hole-nosilk
- SW21: renamed from SW20; footprint Keebio-Parts:Hybrid_PCB_100H_Dual_hole -> Keebio-Parts:Hybrid_PCB_100H_Dual_hole-nosilk
- SW22: renamed from SW21; footprint Keebio-Parts:Hybrid_PCB_100H_Dual_hole -> Keebio-Parts:Hybrid_PCB_100H_Dual_hole-nosilk
- SW23: renamed from SW22; footprint Keebio-Parts:Hybrid_PCB_100H_Dual_hole -> Keebio-Parts:Hybrid_PCB_100H_Dual_hole-nosilk
- SW24: renamed from SW23; footprint Keebio-Parts:Hybrid_PCB_100H_Dual_hole -> Keebio-Parts:Hybrid_PCB_100H_Dual_hole-nosilk
- SW25: renamed from SW24; footprint Keebio-Parts:Hybrid_PCB_100H_Dual_hole -> Keebio-Parts:Hybrid_PCB_100H_Dual_hole-nosilk
- SW26: renamed from SW25; footprint Keebio-Parts:Hybrid_PCB_100H_Dual_hole -> Keebio-Parts:Hybrid_PCB_100H_Dual_hole-nosilk
- moved D21 89.4 mm to (195.3, 138.1), turned to 0 degrees
- moved D22 74.2 mm to (195.3, 138.1)
- moved D16 73.4 mm to (157.2, 128.6), turned to 0 degrees
- moved U1 69.9 mm to (214.3, 76.2)
- moved H3 66.2 mm to (76.2, 85.7)
- moved D24 64.0 mm to (90.5, 95.2), turned to 270 degrees
- moved D25 64.0 mm to (90.5, 114.3), turned to 270 degrees
- moved D23 61.1 mm to (90.5, 76.2), turned to 270 degrees
- moved SW3 60.5 mm to (66.7, 114.3)
- moved H4 59.8 mm to (81.0, 119.1)
- moved D9 59.1 mm to (66.7, 123.8)
- moved D17 57.2 mm to (157.2, 128.6)
- moved D29 57.0 mm to (109.5, 76.2), turned to 270 degrees
- moved D30 57.0 mm to (109.5, 95.2), turned to 270 degrees
- moved D31 57.0 mm to (109.5, 114.3), turned to 270 degrees
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- renumbered D11 to D9
Connections:
- D12 pad 4: Net-(D12-Pad4) -> Net-(D10-Pad2)
- D16 pad 1: /R1 -> VCC
- D16 pad 2: Net-(D13-Pad2) -> Net-(D16-Pad2)
- D17 pad 1: /R2 -> VCC
- D17 pad 2: Net-(D14-Pad2) -> Net-(D17-Pad2)
- D21 pad 1: /R1 -> VCC
- D22 pad 1: /R2 -> VCC
- D23 pad 1: /R3 -> /R1
- D24 pad 1: /R1 -> /R2
- D24 pad 2: Net-(D21-Pad2) -> Net-(D24-Pad2)
- D25 pad 1: /R2 -> /R3
- D25 pad 2: Net-(D22-Pad2) -> Net-(D25-Pad2)
- D8 pad 2: Net-(D12-Pad4) -> Net-(D10-Pad4)
- SW4 pad 2: Net-(D21-Pad2) -> Net-(D23-Pad2)
- SW5 pad 2: Net-(D22-Pad2) -> Net-(D24-Pad2)
- SW6 pad 2: Net-(D23-Pad2) -> Net-(D25-Pad2)
