File: pcb/indigo.sch (KiCad schematic (older format))
At the start: 50 parts

Commit message: pcb started
Parts:
- removed D? (x25): D, symbol Device:D
- removed SW? (x7): SW_Push, symbol Switch:SW_Push
- added D1, D11, D12, D19, D2, D20, D27, D28, D29, D3, D30, D4, D5, D6, D7, D8: WS2812B, LED_SMD:LED_WS2812B_PLCC4_5.0x5.0mm_P3.2mm, symbol LED:WS2812B
- added D13, D14, D15, D16, D17, D18, D21, D22, D23, D24, D25, D26, D31, D32, D33, D34, D35, D36, D37, D38, D39, D40, D41, D42, D43, D44, D45, D46, D47, D48, D49, D50, D51, D52, D53, D54, D55, D56, D57, D58, D59, D60, D61, D62, D63, D64, D65, D66, D67, D68: D, Keebio-Parts:Diode-Hybrid-Back, symbol Device:D
- added H1, H2, H3, H4: MountingHole, keyboard_parts:HOLE_M3, symbol Mechanical:MountingHole
- added SW1, SW2, SW22, SW23, SW24, SW25, SW3: SW_Push, Keebio-Parts:Hybrid_PCB_100H_Dual_hole, symbol Switch:SW_Push
- added U1: ProMicro, promicro:ProMicro, symbol promicro:ProMicro
- SW10, SW11, SW12, SW13, SW14, SW15, SW16, SW17, SW18, SW19, SW20, SW21, SW4, SW5, SW6, SW7, SW8, SW9: renamed from SW?; footprint (none) -> Keebio-Parts:Hybrid_PCB_100H_Dual_hole
Connections:
- net C2: now reaches SW6.1
- net C2: now also SW4.1, SW5.1, U1.12 (B5)
- net at SW6.2: now also D23.2 (A), D26.2 (A)
- net at SW5.2: now also D22.2 (A), D25.2 (A)
- net at SW4.2: now also D21.2 (A), D24.2 (A)
- net C3: now reaches SW9.1
- net C3: now also SW7.1, SW8.1, U1.13 (B6)
- net at SW9.2: now also D33.2 (A), D36.2 (A)
- net at SW8.2: now also D32.2 (A), D35.2 (A)
- net at SW7.2: now also D31.2 (A), D34.2 (A)
- net C4: now reaches SW13.1
- net C4: now also SW10.1, SW11.1, SW12.1, U1.14 (B2)
- net at SW13.2: now also D40.2 (A), D44.2 (A)
- net at SW12.2: now also D39.2 (A), D43.2 (A)
- net at SW11.2: now also D38.2 (A), D42.2 (A)
- net at SW10.2: now also D37.2 (A), D41.2 (A)
- net C5: now reaches SW17.1
- net C5: now also SW14.1, SW15.1, SW16.1, U1.15 (B3)
- net at SW17.2: now also D48.2 (A), D52.2 (A)
- net at SW16.2: now also D47.2 (A), D51.2 (A)
- net at SW15.2: now also D46.2 (A), D50.2 (A)
- net at SW14.2: now also D45.2 (A), D49.2 (A)
- net C6: now reaches SW21.1
- net C6: now also SW18.1, SW19.1, SW20.1, U1.16 (B1)
- net at SW21.2: now also D56.2 (A), D60.2 (A)
- net at SW20.2: now also D55.2 (A), D59.2 (A)
- net at SW19.2: now also D54.2 (A), D58.2 (A)
- net at SW18.2: now also D53.2 (A), D57.2 (A)
- new net: D64.2 (A), D68.2 (A), SW25.2
- new net: D63.2 (A), D67.2 (A), SW24.2
- new net: D62.2 (A), D66.2 (A), SW23.2
- new net: D61.2 (A), D65.2 (A), SW22.2
- new net: D15.2 (A), D18.2 (A), SW3.2
- new net: D14.2 (A), D17.2 (A), SW2.2
- new net: D13.2 (A), D16.2 (A), SW1.2
- new net: D1.2 (DOUT), D3.4 (DIN)
- new net: D3.2 (DOUT), D5.4 (DIN)
- new net: D5.2 (DOUT), D7.4 (DIN)
- new net: D11.4 (DIN), D7.2 (DOUT)
- new net: D11.2 (DOUT), D19.4 (DIN)
- new net: D19.2 (DOUT), D27.4 (DIN)
- new net: D2.2 (DOUT), D4.4 (DIN)
- new net: D4.2 (DOUT), D6.4 (DIN)
- new net: D6.2 (DOUT), D8.4 (DIN)
- new net: D12.4 (DIN), D8.2 (DOUT)
- new net: D12.2 (DOUT), D20.4 (DIN)
- new net: D20.2 (DOUT), D28.4 (DIN)
- new net: D27.2 (DOUT), D29.4 (DIN)
- new net: D28.2 (DOUT), D30.4 (DIN)
- new net C1: SW1.1, SW2.1, SW3.1, U1.11 (B4)
- new net C7: SW22.1, SW23.1, SW24.1, SW25.1, U1.17 (F7)
- new net GND: D1.3 (VSS), D11.3 (VSS), D12.3 (VSS), D19.3 (VSS), D2.3 (VSS), D20.3 (VSS), D27.3 (VSS), D28.3 (VSS), D29.3 (VSS), D3.3 (VSS), D30.3 (VSS), D4.3 (VSS), D5.3 (VSS), D6.3 (VSS), D7.3 (VSS), D8.3 (VSS), U1.23 (GND), U1.3 (GND), U1.4 (GND)
- new net LED_PIN: D1.4 (DIN), D2.4 (DIN), U1.20 (F4)
- new net R1: D13.1 (K), D16.1 (K), D21.1 (K), D24.1 (K), D31.1 (K), D34.1 (K), D37.1 (K), D41.1 (K), D45.1 (K), D49.1 (K), D53.1 (K), D57.1 (K), D61.1 (K), D65.1 (K), U1.7 (D4)
- new net R2: D14.1 (K), D17.1 (K), D22.1 (K), D25.1 (K), D32.1 (K), D35.1 (K), D38.1 (K), D42.1 (K), D46.1 (K), D50.1 (K), D54.1 (K), D58.1 (K), D62.1 (K), D66.1 (K), U1.8 (C6)
- new net R3: D15.1 (K), D18.1 (K), D23.1 (K), D26.1 (K), D33.1 (K), D36.1 (K), D39.1 (K), D43.1 (K), D47.1 (K), D51.1 (K), D55.1 (K), D59.1 (K), D63.1 (K), D67.1 (K), U1.9 (D7)
- new net R4: D40.1 (K), D44.1 (K), D48.1 (K), D52.1 (K), D56.1 (K), D60.1 (K), D64.1 (K), D68.1 (K), U1.10 (E6)
- new net VCC: D1.1 (VDD), D11.1 (VDD), D12.1 (VDD), D19.1 (VDD), D2.1 (VDD), D20.1 (VDD), D27.1 (VDD), D28.1 (VDD), D29.1 (VDD), D3.1 (VDD), D30.1 (VDD), D4.1 (VDD), D5.1 (VDD), D6.1 (VDD), D7.1 (VDD), D8.1 (VDD), U1.21 (VCC)

Commit message: pcb, features
Parts:
- removed D16, D17, D18, D24, D25, D26, D34, D35, D36, D41, D42, D43, D44, D49, D50, D51, D52, D57, D58, D59, D60, D65, D66, D67, D68: D, Keebio-Parts:Diode-Hybrid-Back, symbol Device:D
- added D32: D, Keebio-Parts:Diode-dual, symbol Device:D
- added J1: Conn_01x04, Connector_PinHeader_2.54mm:PinHeader_1x04_P2.54mm_Vertical, symbol Connector_Generic:Conn_01x04
- added R1, R3: R, Keebio-Parts:Resistor-Hybrid, symbol Device:R
- added R2, R4: R, Keebio-Parts:Resistor-Hybrid-Back, symbol Device:R
- added SW10: SW_Push, Keebio-Parts:Hybrid_PCB_100H_Dual_hole-nosilk, symbol Switch:SW_Push
- D13, D14, D15, D37, D38, D39, D40, D45, D46, D47, D48, D53, D54, D55, D56, D61, D62, D63, D64: footprint Keebio-Parts:Diode-Hybrid-Back -> Keebio-Parts:Diode-dual
- D23: renamed from D21; footprint Keebio-Parts:Diode-Hybrid-Back -> Keebio-Parts:Diode-dual
- D24: renamed from D22; footprint Keebio-Parts:Diode-Hybrid-Back -> Keebio-Parts:Diode-dual
- D25: renamed from D23; footprint Keebio-Parts:Diode-Hybrid-Back -> Keebio-Parts:Diode-dual
- D29: renamed from D31; footprint Keebio-Parts:Diode-Hybrid-Back -> Keebio-Parts:Diode-dual
- D30: renamed from D32; footprint Keebio-Parts:Diode-Hybrid-Back -> Keebio-Parts:Diode-dual
- D31: renamed from D33; footprint Keebio-Parts:Diode-Hybrid-Back -> Keebio-Parts:Diode-dual
- SW1, SW2, SW3, SW4, SW5, SW6, SW7, SW8, SW9: footprint Keebio-Parts:Hybrid_PCB_100H_Dual_hole -> Keebio-Parts:Hybrid_PCB_100H_Dual_hole-nosilk
- SW11: renamed from SW10; footprint Keebio-Parts:Hybrid_PCB_100H_Dual_hole -> Keebio-Parts:Hybrid_PCB_100H_Dual_hole-nosilk
- SW12: renamed from SW11; footprint Keebio-Parts:Hybrid_PCB_100H_Dual_hole -> Keebio-Parts:Hybrid_PCB_100H_Dual_hole-nosilk
- SW13: renamed from SW12; footprint Keebio-Parts:Hybrid_PCB_100H_Dual_hole -> Keebio-Parts:Hybrid_PCB_100H_Dual_hole-nosilk
- SW14: renamed from SW13; footprint Keebio-Parts:Hybrid_PCB_100H_Dual_hole -> Keebio-Parts:Hybrid_PCB_100H_Dual_hole-nosilk
- SW15: renamed from SW14; footprint Keebio-Parts:Hybrid_PCB_100H_Dual_hole -> Keebio-Parts:Hybrid_PCB_100H_Dual_hole-nosilk
- SW16: renamed from SW15; footprint Keebio-Parts:Hybrid_PCB_100H_Dual_hole -> Keebio-Parts:Hybrid_PCB_100H_Dual_hole-nosilk
- SW17: renamed from SW16; footprint Keebio-Parts:Hybrid_PCB_100H_Dual_hole -> Keebio-Parts:Hybrid_PCB_100H_Dual_hole-nosilk
- SW18: renamed from SW17; footprint Keebio-Parts:Hybrid_PCB_100H_Dual_hole -> Keebio-Parts:Hybrid_PCB_100H_Dual_hole-nosilk
- SW19: renamed from SW18; footprint Keebio-Parts:Hybrid_PCB_100H_Dual_hole -> Keebio-Parts:Hybrid_PCB_100H_Dual_hole-nosilk
- SW20: renamed from SW19; footprint Keebio-Parts:Hybrid_PCB_100H_Dual_hole -> Keebio-Parts:Hybrid_PCB_100H_Dual_hole-nosilk
- SW21: renamed from SW20; footprint Keebio-Parts:Hybrid_PCB_100H_Dual_hole -> Keebio-Parts:Hybrid_PCB_100H_Dual_hole-nosilk
- SW22: renamed from SW21; footprint Keebio-Parts:Hybrid_PCB_100H_Dual_hole -> Keebio-Parts:Hybrid_PCB_100H_Dual_hole-nosilk
- SW23: renamed from SW22; footprint Keebio-Parts:Hybrid_PCB_100H_Dual_hole -> Keebio-Parts:Hybrid_PCB_100H_Dual_hole-nosilk
- SW24: renamed from SW23; footprint Keebio-Parts:Hybrid_PCB_100H_Dual_hole -> Keebio-Parts:Hybrid_PCB_100H_Dual_hole-nosilk
- SW25: renamed from SW24; footprint Keebio-Parts:Hybrid_PCB_100H_Dual_hole -> Keebio-Parts:Hybrid_PCB_100H_Dual_hole-nosilk
- SW26: renamed from SW25; footprint Keebio-Parts:Hybrid_PCB_100H_Dual_hole -> Keebio-Parts:Hybrid_PCB_100H_Dual_hole-nosilk
- renumbered D12 to D10, D19 to D11, D20 to D12, D27 to D16, D28 to D17, D29 to D21, D30 to D22, D11 to D9
Connections:
- net C3: now also SW10.1
- net GND: now also J1.4 (Pin_4), R1.2, R2.2, R3.2, R4.2
- net R4: now also D32.1 (K)
- net VCC: now also J1.1 (Pin_1)
- net at U1.5 (SCL): now also J1.2 (Pin_2), R3.1, R4.1
- net at U1.6 (SDA): now also J1.3 (Pin_3), R1.1, R2.1
- new net: D32.2 (A), SW10.2
Other:
- moved on the sheet: U1
